Commit message: ar3-platform: real AR3 meshes from ongdexter/ar3_core
Swap the hand-built cylinder placeholder for the CAD-derived AR3
robot description from the ar3_core community package (MIT
licensed; copyright 2021 Dexter Ong).

Asset organization:
- public/ar3-meshes/*.STL: visual + collision meshes (2.6 MB total).
- public/ar3.urdf: rewritten description.
  * package://ar3_description/meshes/ paths → /ar3-meshes/.
  * Six joints changed from "continuous" to "revolute" with
    explicit AR3 firmware limits — ikpy and the slider UI both
    need bounded ranges.
- public/ar3-cylinders.urdf: prior URDF preserved as a fallback
  for debugging mesh/transform issues.
- public/ar3-meshes/ATTRIBUTION.md: source, license, and the two
  local edits documented.

Code adapted to match the upstream naming convention:
- Joint names joint1..joint6 → joint_1..joint_6, link6 → link_6.
  Centralized in Viewer.tsx as JOINT_NAMES / TCP_LINK constants
  rather than scattered f-strings.
- Slider + IK-clamping joint limits updated to the URDF's new
  values (store.ts + sidecar/server.py kept in lockstep).
- Camera home moved slightly and the reach dome bumped to 0.72 m
  to fit the AR3's actual envelope. Shoulder height unchanged.

Verified end-to-end: sidecar loads the new chain, FK home reports
TCP at (-0.007, -0.170, 0.694) in URDF coords, IK converges with
~0 mm residual on reachable targets and fails gracefully on far
ones with no pipeline jam.

https://claude.ai/code/session_01JPszr47TmwRsVUMxfM9Y9k

File: ar3-platform/public/ar3.urdf (robot description, URDF)
Before this commit: robot ar3, 7 links, 6 joints
Links:
- removed link link1
- removed link link2
- removed link link3
- removed link link4
- removed link link5
- removed link link6
- added link link_1, mass 0.88065; collision mesh filename=/ar3-meshes/link_1.STL; visual mesh filename=/ar3-meshes/link_1.STL
- added link link_2, mass 0.57738; collision mesh filename=/ar3-meshes/link_2.STL; visual mesh filename=/ar3-meshes/link_2.STL
- added link link_3, mass 0.1787; collision mesh filename=/ar3-meshes/link_3.STL; visual mesh filename=/ar3-meshes/link_3.STL
- added link link_4, mass 0.34936; collision mesh filename=/ar3-meshes/link_4.STL; visual mesh filename=/ar3-meshes/link_4.STL
- added link link_5, mass 0.11562; collision mesh filename=/ar3-meshes/link_5.STL; visual mesh filename=/ar3-meshes/link_5.STL
- added link link_6, mass 0.013863; collision mesh filename=/ar3-meshes/link_6.STL; visual mesh filename=/ar3-meshes/link_6.STL
- link base_link: mass None -> 0.7102; geometry collision mesh filename=/ar3-meshes/base_link.STL; visual mesh filename=/ar3-meshes/base_link.STL
Joints:
- removed joint joint1
- removed joint joint2
- removed joint joint3
- removed joint joint4
- removed joint joint5
- removed joint joint6
- added joint joint_1: type revolute, parent base_link, child link_1, origin xyz=0 0 0.003445 rpy=3.1416 -1.0248E-21 -1.6736E-05, axis 0 0 1, limit lower=-2.97 upper=2.97 effort=10 velocity=2
- added joint joint_2: type revolute, parent link_1, child link_2, origin xyz=0 0.064146 -0.16608 rpy=1.5708 0.5236 -1.5708, axis 0 0 -1, limit lower=-1.75 upper=1.75 effort=10 velocity=2
- added joint joint_3: type revolute, parent link_2, child link_3, origin xyz=0.1525 -0.26414 0 rpy=3.3431E-16 -1.4164E-16 -1.4953816339, axis 0 0 -1, limit lower=-2.4 upper=2.4 effort=10 velocity=2
- added joint joint_4: type revolute, parent link_3, child link_4, origin xyz=0 0 0.00675 rpy=1.5708 -1.2554 -1.5708, axis 0 0 -1, limit lower=-2.88 upper=2.88 effort=10 velocity=2
- added joint joint_5: type revolute, parent link_4, child link_5, origin xyz=0 0 -0.22225 rpy=3.1416 0 -2.8262, axis -1 0 0, limit lower=-1.83 upper=1.83 effort=10 velocity=2
- added joint joint_6: type revolute, parent link_5, child link_6, origin xyz=-0.000294 0 0.02117 rpy=0 0 3.1416, axis 0 0 1, limit lower=-2.71 upper=2.71 effort=10 velocity=2

Commit message: ar3-platform: fix double-slash in mesh URLs
URDFLoader auto-sets workingPath to the base URL of the .urdf
(`/`), then prepends it to every mesh filename. With our absolute
paths `/ar3-meshes/foo.STL` that produced `//ar3-meshes/foo.STL`,
which the browser parses as a protocol-relative URL — `ar3-meshes`
becomes the hostname and DNS resolution fails (ERR_NAME_NOT_RESOLVED).

Make mesh paths in ar3.urdf relative (`ar3-meshes/foo.STL`); they
now concatenate cleanly with the auto-detected workingPath.

https://claude.ai/code/session_01JPszr47TmwRsVUMxfM9Y9k

File: ar3-platform/public/ar3.urdf (robot description, URDF)
Before this commit: robot ar3, 7 links, 6 joints
Links:
- link base_link: geometry collision mesh filename=ar3-meshes/base_link.STL; visual mesh filename=ar3-meshes/base_link.STL
- link link_1: geometry collision mesh filename=ar3-meshes/link_1.STL; visual mesh filename=ar3-meshes/link_1.STL
- link link_2: geometry collision mesh filename=ar3-meshes/link_2.STL; visual mesh filename=ar3-meshes/link_2.STL
- link link_3: geometry collision mesh filename=ar3-meshes/link_3.STL; visual mesh filename=ar3-meshes/link_3.STL
- link link_4: geometry collision mesh filename=ar3-meshes/link_4.STL; visual mesh filename=ar3-meshes/link_4.STL
- link link_5: geometry collision mesh filename=ar3-meshes/link_5.STL; visual mesh filename=ar3-meshes/link_5.STL
- link link_6: geometry collision mesh filename=ar3-meshes/link_6.STL; visual mesh filename=ar3-meshes/link_6.STL
